File: interactive-jack-o-lantern/src/jack-o-lantern_schematic.sch (EAGLE design)
At the start: 13 parts, among them Q1 S9013

Commit message: Updated instructions with illustrations + added complete circuit frizting
Parts:
- removed D2: (no value), SparkFun-DiscreteSemi:DIODEPTH
- added D3: (no value), SparkFun-LED:WS2812B
- D1: device SparkFun-LED:WS2812B -> SparkFun-DiscreteSemi:DIODEPTH
Connections:
- net D2: now also D3.DIN; no longer D1.DIN
- net GND: now also D1.A, D3.VSS; no longer D1.VSS, D2.A
- net VBAT: now also D1.C, D3.VDD; no longer D1.VDD, D2.C
Changed lines of the file:
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@@
 <part name="U$1" library="Spark" deviceset="SPARK_CORE" device="CORE"/>
 <part name="FRAME1" library="microbuilder" deviceset="FRAME_A4" device=""/>
-<part name="D1" library="SparkFun-LED" deviceset="WS2812B" device=""/>
-<part name="D2" library="SparkFun-DiscreteSemi" deviceset="DIODE" device="PTH"/>
+<part name="D3" library="SparkFun-LED" deviceset="WS2812B" device=""/>
+<part name="D1" library="SparkFun-DiscreteSemi" deviceset="DIODE" device="PTH"/>
 <part name="J_ULTRASONIC_1" library="Ultrasonic Sensor HC-SR04" deviceset="HC-SR04" device=""/>
 <part name="JP1" library="SparkFun-Connectors" deviceset="M05" device="PTH"/>
@@
 <instance part="U$1" gate="G$1" x="78.74" y="124.46"/>
 <instance part="FRAME1" gate="G$1" x="0" y="0"/>
-<instance part="D1" gate="G$1" x="208.28" y="60.96"/>
-<instance part="D2" gate="G$1" x="220.98" y="154.94" smashed="yes" rot="R180">
+<instance part="D3" gate="G$1" x="208.28" y="60.96" smashed="yes">
+<attribute name="VALUE" x="205.74" y="53.34" size="1.778" layer="96"/>
+</instance>
+<instance part="D1" gate="G$1" x="220.98" y="154.94" smashed="yes" rot="R180">
 <attribute name="NAME" x="221.234" y="158.7754" size="1.778" layer="95" rot="R180"/>
 <attribute name="VALUE" x="218.44" y="157.2514" size="1.778" layer="96" rot="R180"/>
@@
 </segment>
 <segment>
-<pinref part="D1" gate="G$1" pin="VSS"/>
+<pinref part="D3" gate="G$1" pin="VSS"/>
 <pinref part="GND5" gate="1" pin="GND"/>
 <wire x1="226.06" y1="58.42" x2="233.68" y2="58.42" width="0.1524" layer="91"/>
@@
 <wire x1="233.68" y1="154.94" x2="226.06" y2="154.94" width="0.1524" layer="91"/>
 <wire x1="226.06" y1="154.94" x2="226.06" y2="157.48" width="0.1524" layer="91"/>
-<pinref part="D2" gate="G$1" pin="A"/>
+<pinref part="D1" gate="G$1" pin="A"/>
 <wire x1="223.52" y1="154.94" x2="226.06" y2="154.94" width="0.1524" layer="91"/>
 <junction x="226.06" y="154.94"/>
@@
 </segment>
 <segment>
-<pinref part="D1" gate="G$1" pin="DIN"/>
+<pinref part="D3" gate="G$1" pin="DIN"/>
 <wire x1="226.06" y1="66.04" x2="236.22" y2="66.04" width="0.1524" layer="91"/>
 <label x="233.68" y="66.04" size="1.778" layer="95"/>
@@
 <segment>
 <pinref part="U$4" gate="G$1" pin="VBAT"/>
-<pinref part="D1" gate="G$1" pin="VDD"/>
+<pinref part="D3" gate="G$1" pin="VDD"/>
 <wire x1="195.58" y1="66.04" x2="203.2" y2="66.04" width="0.1524" layer="91"/>
 </segment>
@@
 <pinref part="U$2" gate="G$1" pin="VBAT"/>
 <wire x1="233.68" y1="152.4" x2="215.9" y2="152.4" width="0.1524" layer="91"/>
-<pinref part="D2" gate="G$1" pin="C"/>
+<pinref part="D1" gate="G$1" pin="C"/>
 <wire x1="215.9" y1="152.4" x2="213.36" y2="152.4" width="0.1524" layer="91"/>
 <wire x1="218.44" y1="154.94" x2="215.9" y2="154.94" width="0.1524" layer="91"/>
